File: sch/mini48-keyboard_v2_mx_choc/mini48-keyboard_v2_mx_choc.kicad_pcb (KiCad board)
At the start: 2 copper layers, 232 x 76 mm, 118 parts, among them SW1 SW_Push, SW10 SW_Push, SW11 SW_Push, SW12 SW_Push, SW13 SW_Push, SW14 SW_Push, SW15 SW_Push, SW16 SW_Push, SW17 SW_Push, SW18 SW_Push, SW19 SW_Push, SW2 SW_Push, SW20 SW_Push, SW21 SW_Push, SW22 SW_Push, SW23 SW_Push, SW24 SW_Push, SW25 SW_Push, SW26 SW_Push, SW27 SW_Push, SW28 SW_Push, SW29 SW_Push, SW3 SW_Push, SW30 SW_Push, SW31 SW_Push, SW32 SW_Push, SW33 SW_Push, SW34 SW_Push, SW35 SW_Push, SW36 SW_Push, SW37 SW_Push, SW38 SW_Push, SW39 SW_Push, SW4 SW_Push, SW40 SW_Push, SW41 SW_Push, SW42 SW_Push, SW43 SW_Push, SW44 SW_Push, SW45 SW_Push, SW46 SW_Push, SW47 SW_Push, SW48 SW_Push, SW5 SW_Push, SW6 SW_Push, SW7 SW_Push, SW8 SW_Push, SW9 SW_Push, U1 Pico

Commit message: MXとchocを並列に接続しました。 基板外形を変更中。
Parts:
- added SW49: SW_Push, my_keyswitch:SW_Hotswap_Kailh_MX, F.Cu at (49.0, 64.0)
- added SW50: SW_Push, my_keyswitch:SW_Hotswap_Kailh_MX, F.Cu at (68.0, 64.0)
- added SW51: SW_Push, my_keyswitch:SW_Hotswap_Kailh_MX, F.Cu at (87.0, 64.0)
- added SW52: SW_Push, my_keyswitch:SW_Hotswap_Kailh_MX, F.Cu at (106.0, 64.0)
- added SW53: SW_Push, my_keyswitch:SW_Hotswap_Kailh_MX, F.Cu at (125.0, 64.0)
- added SW54: SW_Push, my_keyswitch:SW_Hotswap_Kailh_MX, F.Cu at (144.0, 64.0)
- added SW55: SW_Push, my_keyswitch:SW_Hotswap_Kailh_MX, F.Cu at (163.0, 64.0)
- added SW56: SW_Push, my_keyswitch:SW_Hotswap_Kailh_MX, F.Cu at (182.0, 64.0)
- added SW57: SW_Push, my_keyswitch:SW_Hotswap_Kailh_MX, F.Cu at (201.0, 64.0)
- added SW58: SW_Push, my_keyswitch:SW_Hotswap_Kailh_MX, F.Cu at (220.0, 64.0)
- added SW59: SW_Push, my_keyswitch:SW_Hotswap_Kailh_MX, F.Cu at (239.0, 64.0)
- added SW60: SW_Push, my_keyswitch:SW_Hotswap_Kailh_MX, F.Cu at (258.0, 64.0)
- added SW61: SW_Push, my_keyswitch:SW_Hotswap_Kailh_MX, F.Cu at (49.0, 83.0)
- added SW62: SW_Push, my_keyswitch:SW_Hotswap_Kailh_MX, F.Cu at (68.0, 83.0)
- added SW63: SW_Push, my_keyswitch:SW_Hotswap_Kailh_MX, F.Cu at (87.0, 83.0)
- added SW64: SW_Push, my_keyswitch:SW_Hotswap_Kailh_MX, F.Cu at (106.0, 83.0)
- added SW65: SW_Push, my_keyswitch:SW_Hotswap_Kailh_MX, F.Cu at (125.0, 83.0)
- added SW66: SW_Push, my_keyswitch:SW_Hotswap_Kailh_MX, F.Cu at (144.0, 83.0)
- added SW67: SW_Push, my_keyswitch:SW_Hotswap_Kailh_MX, F.Cu at (163.0, 83.0)
- added SW68: SW_Push, my_keyswitch:SW_Hotswap_Kailh_MX, F.Cu at (182.0, 83.0)
- added SW69: SW_Push, my_keyswitch:SW_Hotswap_Kailh_MX, F.Cu at (201.0, 83.0)
- added SW70: SW_Push, my_keyswitch:SW_Hotswap_Kailh_MX, F.Cu at (220.0, 83.0)
- added SW71: SW_Push, my_keyswitch:SW_Hotswap_Kailh_MX, F.Cu at (239.0, 83.0)
- added SW72: SW_Push, my_keyswitch:SW_Hotswap_Kailh_MX, F.Cu at (258.0, 83.0)
- added SW73: SW_Push, my_keyswitch:SW_Hotswap_Kailh_MX, F.Cu at (49.0, 102.0)
- added SW74: SW_Push, my_keyswitch:SW_Hotswap_Kailh_MX, F.Cu at (68.0, 102.0)
- added SW75: SW_Push, my_keyswitch:SW_Hotswap_Kailh_MX, F.Cu at (87.0, 102.0)
- added SW76: SW_Push, my_keyswitch:SW_Hotswap_Kailh_MX, F.Cu at (106.0, 102.0)
- added SW77: SW_Push, my_keyswitch:SW_Hotswap_Kailh_MX, F.Cu at (125.0, 102.0)
- added SW78: SW_Push, my_keyswitch:SW_Hotswap_Kailh_MX, F.Cu at (144.0, 102.0)
- added SW79: SW_Push, my_keyswitch:SW_Hotswap_Kailh_MX, F.Cu at (163.0, 102.0)
- added SW80: SW_Push, my_keyswitch:SW_Hotswap_Kailh_MX, F.Cu at (182.0, 102.0)
- added SW81: SW_Push, my_keyswitch:SW_Hotswap_Kailh_MX, F.Cu at (201.0, 102.0)
- added SW82: SW_Push, my_keyswitch:SW_Hotswap_Kailh_MX, F.Cu at (220.0, 102.0)
- added SW83: SW_Push, my_keyswitch:SW_Hotswap_Kailh_MX, F.Cu at (239.0, 102.0)
- added SW84: SW_Push, my_keyswitch:SW_Hotswap_Kailh_MX, F.Cu at (258.0, 102.0)
- added SW85: SW_Push, my_keyswitch:SW_Hotswap_Kailh_MX, F.Cu at (49.0, 121.0)
- added SW86: SW_Push, my_keyswitch:SW_Hotswap_Kailh_MX, F.Cu at (68.0, 121.0)
- added SW87: SW_Push, my_keyswitch:SW_Hotswap_Kailh_MX, F.Cu at (87.0, 121.0)
- added SW88: SW_Push, my_keyswitch:SW_Hotswap_Kailh_MX, F.Cu at (106.0, 121.0)
- added SW89: SW_Push, my_keyswitch:SW_Hotswap_Kailh_MX, F.Cu at (125.0, 121.0)
- added SW90: SW_Push, my_keyswitch:SW_Hotswap_Kailh_MX, F.Cu at (144.1, 121.0)
- added SW91: SW_Push, my_keyswitch:SW_Hotswap_Kailh_MX, F.Cu at (163.0, 121.0)
- added SW92: SW_Push, my_keyswitch:SW_Hotswap_Kailh_MX, F.Cu at (182.0, 121.0)
- added SW93: SW_Push, my_keyswitch:SW_Hotswap_Kailh_MX, F.Cu at (201.0, 121.0)
- added SW94: SW_Push, my_keyswitch:SW_Hotswap_Kailh_MX, F.Cu at (220.0, 121.0)
- added SW95: SW_Push, my_keyswitch:SW_Hotswap_Kailh_MX, F.Cu at (239.0, 121.0)
- added SW96: SW_Push, my_keyswitch:SW_Hotswap_Kailh_MX, F.Cu at (258.0, 121.0)
- SW1, SW10, SW11, SW12, SW13, SW14, SW15, SW16, SW17, SW18, SW19, SW2, SW20, SW21, SW22, SW23, SW24, SW25, SW26, SW27, SW28, SW29, SW3, SW30, SW31, SW32, SW33, SW34, SW35, SW36, SW37, SW38, SW39, SW4, SW40, SW41, SW42, SW43, SW44, SW45, SW46, SW47, SW48, SW5, SW6, SW7, SW8, SW9: footprint my_keyswitch:CherryMX_MidHeight_Choc_Hotswap_rev1 -> my_keyswitch:SW_Hotswap_Kailh_Choc_V1V2_no_mp
- U1: moved to F.Cu
- moved REF** 70.5 mm to (154.0, 163.0)
- moved U1 63.2 mm to (241.9, 39.1), turned to -90 degrees
- moved REF** 53.6 mm to (131.0, 146.0)
- moved REF** 53.5 mm to (94.0, 146.0)
- moved REF** 52.5 mm to (209.0, 145.0)
- moved REF** 50.7 mm to (176.0, 143.0)
- moved REF** 42.6 mm to (144.0, 170.0)
- moved REF** 39.7 mm to (74.0, 18.0)
- moved REF** 39.6 mm to (113.0, 18.0)
- moved REF** 39.5 mm to (190.0, 18.0)
- moved REF** 39.5 mm to (153.0, 18.0)
- moved REF** 38.5 mm to (229.0, 19.0)
- moved REF** 24.6 mm to (29.0, 151.0)
- moved REF** 24.5 mm to (77.0, 153.0)
- moved REF** 24.5 mm to (116.0, 153.0)
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Routing:
- net /ROW0: track 326.3 -> 16.2 mm
- net /ROW3: track 300.1 -> 16.2 mm
- net /ROW2: track 285.6 -> 16.2 mm
- net /ROW1: track 281.9 -> 16.2 mm
- net /COL0: track 244.9 -> 66.7 mm, vias 1 -> 0
- net /COL1: track 229.5 -> 68.6 mm, vias 1 -> 0
- net /COL2: track 217.8 -> 66.7 mm, vias 1 -> 0
- net /COL3: track 207.6 -> 66.7 mm, vias 1 -> 0
- net /COL4: track 201.6 -> 66.7 mm, vias 1 -> 0
- net /COL5: track 179.9 -> 66.7 mm, vias 1 -> 0
- net /COL11: track 98.6 -> 11.6 mm
- net /COL6: track 130.3 -> 72.2 mm, vias 1 -> 0
- net /COL7: track 113.9 -> 66.7 mm, vias 1 -> 0
- net /COL8: track 108.6 -> 68.6 mm, vias 1 -> 0
- net /COL10: track 67.3 -> 28.9 mm
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Other:
- board size 232 x 76 mm -> 232 x 107 mm
- board text added: "mini48-keyboard v2.0 (MX/CHOC)"
- board text removed: "mini48-keyboard v.2 (MX/CHOC)"

Commit message: 基板上にUSB type-cのコネクタを実装しました。 picoのTPとジャンパ配線します。
Parts:
- removed REF** (x20): MountingHole_2.2mm_M2, MountingHole:MountingHole_2.2mm_M2
- removed REF**: MountingHole_6.4mm_M6, MountingHole:MountingHole_6.4mm_M6
- added H1: MountingHole, my_keyswitch:my_MountingHole_3.2mm_M3, F.Cu at (58.5, 73.5)
- added H10: MountingHole, my_keyswitch:my_MountingHole_3.2mm_M3, F.Cu at (229.5, 92.5)
- added H11: MountingHole, my_keyswitch:my_MountingHole_3.2mm_M3, F.Cu at (248.5, 73.5)
- added H12: MountingHole, my_keyswitch:my_MountingHole_3.2mm_M3, F.Cu at (248.5, 111.5)
- added H2: MountingHole, my_keyswitch:my_MountingHole_3.2mm_M3, F.Cu at (58.5, 111.5)
- added H3: MountingHole, my_keyswitch:my_MountingHole_3.2mm_M3, F.Cu at (77.5, 92.5)
- added H4: MountingHole, my_keyswitch:my_MountingHole_3.2mm_M3, F.Cu at (96.5, 73.5)
- added H5: MountingHole, my_keyswitch:my_MountingHole_3.2mm_M3, F.Cu at (96.5, 111.5)
- added H6: MountingHole, my_keyswitch:my_MountingHole_3.2mm_M3, F.Cu at (115.5, 92.5)
- added H7: MountingHole, my_keyswitch:my_MountingHole_3.2mm_M3, F.Cu at (191.5, 92.5)
- added H8: MountingHole, my_keyswitch:my_MountingHole_3.2mm_M3, F.Cu at (210.5, 73.5)
- added H9: MountingHole, my_keyswitch:my_MountingHole_3.2mm_M3, F.Cu at (210.5, 111.5)
- added J1: 5077CR-16SMC2-BK-TR, usb_c:NELTRON_5077CR-16SMC2-BK-TR, B.Cu at (200.1, 30.4)
- added R1: 5.1k, Resistor_SMD:R_0603_1608Metric, B.Cu at (193.0, 35.0)
- added R2: 5.1k, Resistor_SMD:R_0603_1608Metric, B.Cu at (210.0, 34.0)
- added TP1: TestPoint, TestPoint:TestPoint_Pad_1.5x1.5mm, B.Cu at (208.0, 40.5)
- added TP2: TestPoint, TestPoint:TestPoint_Pad_1.5x1.5mm, B.Cu at (208.0, 37.0)
- added TP3: TestPoint, TestPoint:TestPoint_Pad_1.5x1.5mm, B.Cu at (208.0, 44.0)
- U1: footprint my_pico:pico_no_dbg_th_p0.85 -> my_pico:pico_no_dbg_smd_th_p0.85
Routing:
- net /ROW3: track 16.2 -> 397.2 mm
- net /ROW2: track 16.2 -> 131.9 mm
- net /ROW1: track 16.2 -> 84.9 mm
- net /ROW0: track 16.2 -> 55.2 mm
- net Net-(J1-VBUS-PadA4_B9): track 0.00 -> 24.7 mm, vias 0 -> 3
- net /usb type-c/USB_N: track 0.00 -> 19.6 mm
- net /usb type-c/USB_P: track 0.00 -> 16.1 mm
- net Net-(J1-CC2): track 0.00 -> 9.82 mm
- net Net-(J1-CC1): track 0.00 -> 8.12 mm
Other:
- outline, holes or cut-outs redrawn
- board text added: "DM"
- board text added: "DP"
- board text added: "VBUS"
