File: sch/mini40-keyboard_v2_p17/mini40-keyboard_v2_p17.kicad_pcb (KiCad board)
At the start: 2 copper layers, 175 x 112 mm, 103 parts, among them J1 Conn_01x02, J2 Conn_02x08_Odd_Even, Q1 DMG2301L, SW1 SW_Push, SW10 SW_Push, SW11 SW_Push, SW12 SW_Push, SW13 SW_Push, SW14 SW_Push, SW15 SW_Push, SW16 SW_Push, SW17 SW_Push, SW18 SW_Push, SW19 SW_Push, SW2 SW_Push, SW20 SW_Push, SW21 SW_Push, SW22 SW_Push, SW23 SW_Push, SW24 SW_Push, SW25 SW_Push, SW26 SW_Push, SW27 SW_Push, SW28 SW_Push, SW29 SW_Push, SW3 SW_Push, SW30 SW_Push, SW31 SW_Push, SW32 SW_Push, SW33 SW_Push, SW34 SW_Push, SW35 SW_Push, SW36 SW_Push, SW37 SW_Push, SW38 SW_Push, SW39 SW_Push, SW4 SW_Push, SW40 SW_Push, SW5 SW_Push, SW6 SW_Push, SW7 SW_Push, SW8 SW_Push, SW9 SW_Push, U1 Pico, U2 pimoroni lcd

Commit message: マイコンとしてESP32-S3の使用を検討しています。 Rasberry Pi Pico と ESP32-S3 のどちらかを選択して実装する設計です。 主要部品以外は仮の部品・フットプリントです。
Parts:
- added C1: 10u, Capacitor_SMD:C_0603_1608Metric_Pad1.08x0.95mm_HandSolder, F.Cu at (-22.3, 68.4)
- added C2: 100n, Capacitor_SMD:C_0603_1608Metric_Pad1.08x0.95mm_HandSolder, F.Cu at (-22.3, 70.9)
- added C3: 100n, Capacitor_SMD:C_0603_1608Metric_Pad1.08x0.95mm_HandSolder, F.Cu at (-22.3, 73.4)
- added C4: 1u, Capacitor_SMD:C_0603_1608Metric_Pad1.08x0.95mm_HandSolder, F.Cu at (-22.3, 76.0)
- added C5: 470p, Capacitor_SMD:C_0603_1608Metric_Pad1.08x0.95mm_HandSolder, F.Cu at (-22.3, 78.5)
- added C6: 10n, Capacitor_SMD:C_0603_1608Metric_Pad1.08x0.95mm_HandSolder, F.Cu at (-22.3, 81.0)
- added C7: 15p, Capacitor_SMD:C_0603_1608Metric_Pad1.08x0.95mm_HandSolder, F.Cu at (-22.3, 83.5)
- added C8: 15p, Capacitor_SMD:C_0603_1608Metric_Pad1.08x0.95mm_HandSolder, F.Cu at (-22.3, 86.0)
- added D41: D_Schottky, Diode_SMD:D_SOD-123, F.Cu at (-21.5, 48.7)
- added D42: D_Schottky, Diode_SMD:D_SOD-123, F.Cu at (-21.5, 52.1)
- added D43: D_Schottky, Diode_SMD:D_SOD-123, F.Cu at (-21.5, 55.4)
- added D44: D_TVS, Diode_SMD:D_SOD-123, F.Cu at (-21.5, 58.8)
- added D45: D_TVS, Diode_SMD:D_SOD-123, F.Cu at (-21.5, 62.1)
- added D46: D_TVS, Diode_SMD:D_SOD-123, F.Cu at (-21.5, 65.5)
- added D47: LED, LED_SMD:LED_0603_1608Metric_Pad1.05x0.95mm_HandSolder, F.Cu at (-17.9, 68.5)
- added D48: LED, LED_SMD:LED_0603_1608Metric_Pad1.05x0.95mm_HandSolder, F.Cu at (-17.9, 71.0)
- added D49: LED, LED_SMD:LED_0603_1608Metric_Pad1.05x0.95mm_HandSolder, F.Cu at (-17.9, 73.6)
- added D50: LED, LED_SMD:LED_0603_1608Metric_Pad1.05x0.95mm_HandSolder, F.Cu at (-17.9, 76.2)
- added D51: LED, LED_SMD:LED_0603_1608Metric_Pad1.05x0.95mm_HandSolder, F.Cu at (-17.9, 78.8)
- added D52: LED, LED_SMD:LED_0603_1608Metric_Pad1.05x0.95mm_HandSolder, F.Cu at (-17.9, 81.4)
- added D53: LED, LED_SMD:LED_0603_1608Metric_Pad1.05x0.95mm_HandSolder, F.Cu at (-17.9, 84.0)
- added F1: Polyfuse_Small, Fuse:Fuse_Littelfuse-NANO2-451_453, F.Cu at (-9.94, 19.6)
- added J3: USB_C_Receptacle_USB2.0_16P, Connector_USB:USB_C_Receptacle_XKB_U262-16XN-4BVC11, F.Cu at (-26.5, 22.5)
- added J4: Conn_01x04, Connector_JST:JST_XH_B4B-XH-A_1x04_P2.50mm_Vertical, F.Cu at (-43.4, 20.6)
- added R10: [10M], Resistor_SMD:R_0603_1608Metric, F.Cu at (-56.9, 31.1)
- added R11: 0, Resistor_SMD:R_0603_1608Metric, F.Cu at (-52.9, 18.5)
- added R12: 0, Resistor_SMD:R_0603_1608Metric, F.Cu at (-52.9, 21.0)
- added R13: 1k, Resistor_SMD:R_0603_1608Metric, F.Cu at (-52.9, 23.5)
- added R14: 1k, Resistor_SMD:R_0603_1608Metric, F.Cu at (-52.9, 26.0)
- added R15: 1k, Resistor_SMD:R_0603_1608Metric, F.Cu at (-52.9, 28.5)
- added R16: 1k, Resistor_SMD:R_0603_1608Metric, F.Cu at (-52.9, 31.1)
- added R17: 1k, Resistor_SMD:R_0603_1608Metric, F.Cu at (-48.8, 18.5)
- added R18: 1k, Resistor_SMD:R_0603_1608Metric, F.Cu at (-48.8, 21.0)
- added R19: 1k, Resistor_SMD:R_0603_1608Metric, F.Cu at (-48.8, 23.5)
- added R5: 5.1k, Resistor_SMD:R_0603_1608Metric, F.Cu at (-56.9, 18.5)
- added R6: 5.1k, Resistor_SMD:R_0603_1608Metric, F.Cu at (-56.9, 21.0)
- added R7: 10k, Resistor_SMD:R_0603_1608Metric, F.Cu at (-56.9, 23.5)
- added R8: 0, Resistor_SMD:R_0603_1608Metric, F.Cu at (-56.9, 26.0)
- added R9: 0, Resistor_SMD:R_0603_1608Metric, F.Cu at (-56.9, 28.5)
- added SW41: SW_Push, Button_Switch_SMD:SW_Push_SPST_NO_Alps_SKRK, F.Cu at (-17.4, 19.5)
- added SW42: SW_Push, Button_Switch_SMD:SW_Push_SPST_NO_Alps_SKRK, F.Cu at (-17.4, 23.9)
- added U3: ESP32-S3-WROOM-1, RF_Module:ESP32-S3-WROOM-1, F.Cu at (51.0, 73.2)
- added U4: MIC5219-3.3YM5, Package_TO_SOT_SMD:SOT-23-5, F.Cu at (-11.6, 24.4)
- added Y1: 32k, Crystal:Crystal_SMD_2012-2Pin_2.0x1.2mm_HandSoldering, F.Cu at (-11.9, 28.0)
- moved Q1 0.06 mm to (209.0, 73.0)
Connections:
- net /GPIO10 renamed /COL5
- net /GPIO11 renamed /COL4
- net /GPIO12 renamed /COL3
- net /GPIO13 renamed /COL2
- net /GPIO14 renamed /COL1
- net /GPIO15 renamed /COL0
- net /GPIO16 renamed /DC
- net /GPIO17 renamed /CS_N
- net /GPIO18 renamed /SCLK
- net /GPIO19 renamed /DATA
- net /GPIO2 renamed /ROW3
- net /GPIO20 renamed /LCD_BL
- net /GPIO21 renamed /LCD_TE
- net /GPIO22 renamed /OLED_RESET
- net /GPIO3 renamed /ROW2
- net /GPIO4 renamed /ROW1
- net /GPIO5 renamed /ROW0
- net /GPIO6 renamed /COL9
- net /GPIO7 renamed /COL8
- net /GPIO8 renamed /COL7
- net /GPIO9 renamed /COL6
- net /RUN renamed /LCD_RESET
- net Net-(J1-Pin_1) renamed /VBAT
